Commit message: Fixed point cloud usage and added point cloud visualisation

File: catkin_ws/src/universal_robot/ur_description/urdf/ur5.urdf.xacro (robot description, xacro)
@@ -87,4 +87,17 @@
       </xacro:cylinder_inertial>
     </link>
+	<link name="bumblebee" >
+		<visual>
+			<geometry>
+				<box size="0.1 0.02 0.02"/>
+			</geometry>
+			<origin rpy="0 0 0" xyz="0 0 0"/>
+		</visual>
+	</link>
+	  <joint name="bumblebee_joint" type="fixed">
+		<parent link="base_link"/>
+		<child link="bumblebee"/>
+		<origin rpy="${-pi / 2} 0.0 0.0" xyz="0.0 0.1 0.01"/>
+	  </joint>
     <joint name="${prefix}shoulder_pan_joint" type="revolute">
       <parent link="${prefix}base_link" />

Commit message: Added description files for KasPR.
Also added debug service for arm testing.
This branch is nowhere near ready as it still needs the srdf and other moveIt kinematic files.

File: catkin_ws/src/universal_robot/ur_description/urdf/ur5.urdf.xacro (robot description, xacro)
@@ -87,17 +87,4 @@
       </xacro:cylinder_inertial>
     </link>
-	<link name="bumblebee" >
-		<visual>
-			<geometry>
-				<box size="0.1 0.02 0.02"/>
-			</geometry>
-			<origin rpy="0 0 0" xyz="0 0 0"/>
-		</visual>
-	</link>
-	  <joint name="bumblebee_joint" type="fixed">
-		<parent link="base_link"/>
-		<child link="bumblebee"/>
-		<origin rpy="${-pi / 2} 0.0 0.0" xyz="0.0 0.1 0.01"/>
-	  </joint>
     <joint name="${prefix}shoulder_pan_joint" type="revolute">
       <parent link="${prefix}base_link" />

Commit message: Fixed bumblebee positioning

File: catkin_ws/src/universal_robot/ur_description/urdf/ur5.urdf.xacro (robot description, xacro)
@@ -92,5 +92,5 @@
 				<box size="0.1 0.02 0.02"/>
 			</geometry>
-			<origin rpy="0 0 0" xyz="0 0 0"/>
+			<origin rpy="0.69 0 0" xyz="0 0 0"/>
 		</visual>
 	</link>

Commit message: Fixed point cloud position

File: catkin_ws/src/universal_robot/ur_description/urdf/ur5.urdf.xacro (robot description, xacro)
@@ -92,5 +92,5 @@
 				<box size="0.1 0.02 0.02"/>
 			</geometry>
-			<origin rpy="0.69 0 0" xyz="0 0 0"/>
+			<origin rpy="0.69 0 0" xyz="0.0 0.0 0.0"/>
 		</visual>
 	</link>
@@ -98,5 +98,5 @@
 		<parent link="base_link"/>
 		<child link="bumblebee"/>
-		<origin rpy="${-pi / 2} 0.0 0.0" xyz="0.0 0.1 0.01"/>
+		<origin rpy="${-pi / 2 + 0.69} 0.0 0.0" xyz="-0.16 0.1285 0.0"/>
 	  </joint>
     <joint name="${prefix}shoulder_pan_joint" type="revolute">

Commit message: Improved robot urdf
- Added the robot foundation
- Correctly positioned the stereo camera
- Moved floor and back wall

File: catkin_ws/src/universal_robot/ur_description/urdf/ur5.urdf.xacro (robot description, xacro)
@@ -90,7 +90,10 @@
 		<visual>
 			<geometry>
-				<box size="0.1 0.02 0.02"/>
+				<box size="0.15 0.035 0.045"/>
 			</geometry>
-			<origin rpy="0.69 0 0" xyz="0.0 0.0 0.0"/>
+			<origin rpy="0 0 0" xyz="0.135 0 0"/>
+			<material name="Gold">
+			  <color rgba="1 0.9 0.0 1.0"/>
+			</material>
 		</visual>
 	</link>
@@ -98,5 +101,21 @@
 		<parent link="base_link"/>
 		<child link="bumblebee"/>
-		<origin rpy="${-pi / 2 + 0.69} 0.0 0.0" xyz="-0.16 0.1285 0.0"/>
+		<origin rpy="${-pi / 2 + 0.69} 0.0 0.0" xyz="-0.16 0.1285 -0.035"/>
+	  </joint>
+	<link name="foundation" >
+		<visual>
+			<geometry>
+				<box size="0.245 0.25 0.26"/>
+			</geometry>
+			<origin rpy="0 0 0" xyz="0 -0.055 -0.13"/>
+			<material name="LightGrey">
+			  <color rgba="0.7 0.7 0.7 1.0"/>
+			</material>
+		</visual>
+	</link>
+	  <joint name="foundation_joint" type="fixed">
+		<parent link="base_link"/>
+		<child link="foundation"/>
+		<origin rpy="0 0 0" xyz="0 0 0"/>
 	  </joint>
     <joint name="${prefix}shoulder_pan_joint" type="revolute">

Commit message: Returned the point cloud and raised the table

File: catkin_ws/src/universal_robot/ur_description/urdf/ur5.urdf.xacro (robot description, xacro)
@@ -97,9 +97,15 @@
 			</material>
 		</visual>
+		<collision>
+			<geometry>
+				<box size="0.15 0.035 0.045"/>
+			</geometry>
+			<origin rpy="0 0 0" xyz="0.135 0 0"/>
+		</collision>
 	</link>
 	  <joint name="bumblebee_joint" type="fixed">
 		<parent link="base_link"/>
 		<child link="bumblebee"/>
-		<origin rpy="${-pi / 2 + 0.69} 0.0 0.0" xyz="-0.16 0.1285 -0.035"/>
+		<origin rpy="${-pi / 2} 0.0 0.0" xyz="-0.16 0.1285 0"/>
 	  </joint>
 	<link name="foundation" >

Commit message: Added the end effector to the urdf

File: catkin_ws/src/universal_robot/ur_description/urdf/ur5.urdf.xacro (robot description, xacro)
@@ -87,4 +87,26 @@
       </xacro:cylinder_inertial>
     </link>
+	<link name="end_effector" >
+		<visual>
+			<geometry>
+				<box size="0.075 0.075 0.12"/>
+			</geometry>
+			<origin rpy="0 0 0" xyz="0 0 0.06"/>
+			<material name="White">
+			  <color rgba="1 1 1 1"/>
+			</material>
+		</visual>
+		<collision>
+			<geometry>
+				<box size="0.075 0.075 0.12"/>
+			</geometry>
+			<origin rpy="0 0 0" xyz="0 0 0.06"/>
+		</collision>
+	</link>
+	<joint name="end_effector_joint" type="fixed">
+	<parent link="${prefix}tool0"/>
+	<child link="end_effector"/>
+	<origin rpy="0.0 0.0 0.0" xyz="0 0 0"/>
+	</joint>
 	<link name="bumblebee" >
 		<visual>

Commit message: Fixed table and roof and added missing collision data

File: catkin_ws/src/universal_robot/ur_description/urdf/ur5.urdf.xacro (robot description, xacro)
@@ -141,4 +141,10 @@
 			</material>
 		</visual>
+		<collision>
+			<geometry>
+				<box size="0.245 0.25 0.26"/>
+			</geometry>
+			<origin rpy="0 0 0" xyz="0 -0.055 -0.13"/>
+		</collision>
 	</link>
 	  <joint name="foundation_joint" type="fixed">

Commit message: Angle is 30 degrees again

File: catkin_ws/src/universal_robot/ur_description/urdf/ur5.urdf.xacro (robot description, xacro)
@@ -129,5 +129,5 @@
 		<parent link="base_link"/>
 		<child link="bumblebee"/>
-		<origin rpy="${-pi / 2} 0.0 0.0" xyz="-0.16 0.1285 0"/>
+		<origin rpy="${-pi / 2 + 0.52 - 0.52} 0.0 0.0" xyz="-0.16 0.1285 0"/>
 	  </joint>
 	<link name="foundation" >

Commit message: Fixed various sizes and settings

File: catkin_ws/src/universal_robot/ur_description/urdf/ur5.urdf.xacro (robot description, xacro)
@@ -90,7 +90,7 @@
 		<visual>
 			<geometry>
-				<box size="0.075 0.075 0.12"/>
-			</geometry>
-			<origin rpy="0 0 0" xyz="0 0 0.06"/>
+				<box size="0.1 0.1 0.18"/>
+			</geometry>
+			<origin rpy="0 0 0" xyz="0 0.015 0.09"/>
 			<material name="White">
 			  <color rgba="1 1 1 1"/>
@@ -99,7 +99,7 @@
 		<collision>
 			<geometry>
-				<box size="0.075 0.075 0.12"/>
-			</geometry>
-			<origin rpy="0 0 0" xyz="0 0 0.06"/>
+				<box size="0.1 0.1 0.18"/>
+			</geometry>
+			<origin rpy="0 0 0" xyz="0 0.015 0.091"/>
 		</collision>
 	</link>
@@ -129,5 +129,5 @@
 		<parent link="base_link"/>
 		<child link="bumblebee"/>
-		<origin rpy="${-pi / 2 + 0.52 - 0.52} 0.0 0.0" xyz="-0.16 0.1285 0"/>
+		<origin rpy="${-pi / 2 + 0.52 - 0.69} 0.0 0.0" xyz="-0.06 0.1285 0"/>
 	  </joint>
 	<link name="foundation" >

Commit message: Fixed the point cloud rotation

File: catkin_ws/src/universal_robot/ur_description/urdf/ur5.urdf.xacro (robot description, xacro)
@@ -129,5 +129,5 @@
 		<parent link="base_link"/>
 		<child link="bumblebee"/>
-		<origin rpy="${-pi / 2 + 0.52 - 0.69} 0.0 0.0" xyz="-0.06 0.1285 0"/>
+		<origin rpy="${-pi / 2 + 0.52} 0.0 0.0" xyz="-0.06 0.1285 0"/>
 	  </joint>
 	<link name="foundation" >
